File: FlightController3.brd (EAGLE design)
At the start: 50 x 85 mm, 43 parts, among them T1 BC171B, U1 NUCLEO_L432KC

Commit message: wip
Parts:
- removed C11: NAVBOARD, pinhead:1X04
- removed C6: SBUS, pinhead:1X03
- removed LED1: 5V, led:SML0603
- removed LED2: 3V3, led:SML0603
- removed LED_SCL: (no value), led:SML0603
- removed R12: 110, rcl:M1206
- removed T1: BC171B, transistor:TO92
- removed U$3: AT24C16C, JonasLib:DIL08
- added LED3V: orange, led:SML0603
- added LED5V: green, led:SML0603
- added MF3: BSN20,215, BSN20_215:BSN20_215
- INS1: device 1_Robo-Lib:BNO055-BREAKOUT -> jonas_breakouts:BNO055-BREAKOUT
- JP1: value RESET -> (none); device pinhead:1X02 -> pinhead:1X03
- R10, R11, R9: device rcl:M1206 -> rcl:R0603
- R7, R8: device resistor:M1206 -> rcl:R0603
- U$4: device MPL3115A2:MPL3115A2 -> jonas_breakouts:MPL3115A2
- U1: device NUCLEO:NUCLEO -> jonas_breakouts:NUCLEO
- moved S1 66.3 mm to (32.7, 79.4), turned to 0 degrees
- moved NAV_RX 55.0 mm to (13.0, 80.0), turned to 270 degrees
- moved NAV_TX 54.7 mm to (18.0, 80.0), turned to 270 degrees
- moved U$1 49.3 mm to (-27.9, 61.0)
- moved R10 48.1 mm to (13.0, 76.0), turned to 270 degrees
- moved R9 47.8 mm to (18.0, 76.0), turned to 270 degrees
- moved C2 41.9 mm to (47.6, 15.0), flipped to the bottom
- moved R1 33.5 mm to (2.98, 68.6), turned to 90 degrees
- moved C18 33.4 mm to (18.0, 58.0), turned to 180 degrees
- moved C3 32.1 mm to (42.5, 15.0), flipped to the bottom
- moved C15 29.3 mm to (33.0, 43.0), turned to 0 degrees
- moved U$2 28.5 mm to (-15.2, 61.0), flipped to the top
- moved R2 26.8 mm to (3.00, 59.0), turned to 90 degrees
- moved SJ1 24.8 mm to (3.00, 63.5), turned to 270 degrees
- moved R5 23.2 mm to (20.0, 62.0)
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Connections:
- removed net N$7: LED_SCL.A, R12.1
- net !RST: no longer JP1.1
- net !SBUS: now also MF3.3; no longer T1.3
- net +5V: now also JP1.2; no longer C11.1, C6.2, R12.2, U$3.8
- net GND: now also JP1.3, LED3V.C, LED5V.C, MF3.2; no longer C11.2, C6.3, JP1.2, LED1.C, LED2.C, T1.1, U$3.4, U$3.7
- net N$1: now also MF3.1; no longer T1.2
- net N$2: now also LED3V.A; no longer LED2.A
- net N$3: now also LED5V.A; no longer LED1.A
- net NAVBOARD_RX: no longer C11.4
- net NAVBOARD_TX: no longer C11.3
- net SBUS: now also JP1.1; no longer C6.1
- net SCL5V: no longer LED_SCL.C, U$3.6
- net SDA5V: no longer U$3.5
Routing:
- net SCL5V: track 120.0 -> 62.2 mm, vias 2 -> 0
- net SBUS: track 33.6 -> 88.7 mm, vias 2 -> 1
- net SDA5V: track 108.1 -> 56.6 mm, vias 1 -> 0
- net !RST: track 88.3 -> 47.0 mm, vias 4 -> 1
- net N$10: track 34.5 -> 4.62 mm, vias 2 -> 0
- net NAVBOARD_TX: track 51.2 -> 28.9 mm
- net +5V: track 177.8 -> 158.3 mm, vias 2 -> 1
- net +3V3: track 145.2 -> 129.7 mm, vias 6 -> 4
- net D13: track 32.7 -> 20.4 mm, vias 1 -> 0
- net PPM_MOTOR: track 32.1 -> 44.0 mm, vias 0 -> 2
- net PPM_V_TAIL_L: track 37.2 -> 48.5 mm
- net A0: track 40.5 -> 29.7 mm, vias 2 -> 0
- net SCL: track 29.5 -> 19.1 mm
- net D11: track 29.0 -> 18.8 mm
- net D10: track 32.6 -> 22.4 mm
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Other:
- board text removed: "P.L.A.N.E. v1.0"
